File: RPi-I2C-LevelShifter.brd (EAGLE design)
At the start: 14.9 x 29.2 mm, 8 parts, among them Q1 2N7002, Q2 2N7002

Commit message: fixed error
Parts:
- moved SV1 1.27 mm to (8.89, 24.1)
- moved SV2 1.27 mm to (8.89, 5.08)
- moved Q1 1.27 mm to (5.08, 17.8)
- moved R1 1.27 mm to (5.08, 11.4)
- moved R2 1.27 mm to (5.08, 14.0)
Connections:
- new net P10: SV1.10, SV2.10
- new net P7: SV1.7, SV2.7
- new net P8: SV1.8, SV2.8
- new net P9: SV1.9, SV2.9
- new net SCL_OUT: Q1.3, R1.1, SV2.6
- new net SDA_OUT: Q2.3, R34.1, SV2.4
- net SCL_IN: now also Q1.2, R2.2, SV1.6; no longer Q2.2, Q2.3, R34.1, R35.2, SV1.4, SV2.4
- net SDA_IN: now also Q2.2, R35.2, SV1.4; no longer Q1.2, Q1.3, R1.1, R2.2, SV1.6, SV2.6
Routing:
- net SCL_OUT: track 0.00 -> 45.9 mm
- net P7: track 0.00 -> 30.6 mm
- net SDA_IN: track 40.8 -> 14.6 mm
- net P9: track 0.00 -> 25.3 mm
- net +3V3: track 31.5 -> 55.4 mm
- net SCL_IN: track 32.1 -> 10.2 mm
- net P8: track 0.00 -> 20.8 mm
- net SDA_OUT: track 0.00 -> 20.6 mm
- net P10: track 0.00 -> 20.2 mm
- net +5V: track 48.7 -> 30.1 mm
- net GND: track 44.6 -> 39.1 mm
Other:
- board size 14.9 x 29.2 mm -> 17.4 x 29.2 mm

Commit message: optimized layout
Parts:
- moved Q2 7.62 mm to (3.81, 17.8)
- moved R34 7.62 mm to (3.81, 11.4)
- moved R35 7.62 mm to (3.81, 14.0)
- moved Q1 5.08 mm to (10.2, 17.8)
- moved R1 5.08 mm to (10.2, 11.4)
- moved R2 5.08 mm to (10.2, 14.0)
- moved SV1 1.27 mm to (7.62, 24.1)
- moved SV2 1.27 mm to (7.62, 5.08)
Routing:
- net SCL_OUT: track 45.9 -> 21.3 mm
- net +5V: track 30.1 -> 53.5 mm
- net P8: track 20.8 -> 37.3 mm
- net +3V3: track 55.4 -> 39.7 mm
- net GND: track 39.1 -> 24.1 mm
- net P7: track 30.6 -> 21.1 mm
- net P9: track 25.3 -> 19.8 mm
- net SDA_IN: track 14.6 -> 9.14 mm
- net P10: track 20.2 -> 25.6 mm
- net SDA_OUT: track 20.6 -> 18.7 mm
- net SCL_IN: track 10.2 -> 10.7 mm
Other:
- board size 17.4 x 29.2 mm -> 16.2 x 29.2 mm

Commit message: added simulation; improved layout
Parts:
- moved R34 6.48 mm to (5.08, 17.8), turned to 0 degrees
- moved R1 6.35 mm to (10.2, 17.8), turned to 180 degrees
- moved Q2 4.02 mm to (5.08, 14.0)
- moved R35 4.02 mm to (5.08, 10.2)
- moved Q1 3.81 mm to (10.2, 14.0)
- moved R2 3.81 mm to (10.2, 10.2)
Routing:
- net +5V: track 53.5 -> 35.6 mm
- net GND: track 24.1 -> 41.2 mm
- net SCL_OUT: track 21.3 -> 15.5 mm
- net P10: track 25.6 -> 20.3 mm
- net P8: track 37.3 -> 32.2 mm
- net SDA_IN: track 9.14 -> 14.0 mm
- net SCL_IN: track 10.7 -> 15.0 mm
- net +3V3: track 39.7 -> 36.7 mm
- net P7: track 21.1 -> 21.7 mm
